Commit message: lidar addition

File: description/properties.xacro (robot description, xacro)
@@ -14,3 +14,6 @@
         <color rgba= "0 0 0 1"/>
     </material>
+    <material name="red">
+        <color rgba= "1 0 0 1"/>
+    </material>
 </robot>

File: description/robot.urdf.xacro (robot description, xacro)
@@ -6,3 +6,4 @@
     <xacro:include filename="robot_core.xacro"/>
     <xacro:include filename="gazebo_control.xacro"/>
+    <xacro:include filename="lidar.xacro"/>
 </robot>
