Commit message: mapping_SLAM

File: description/robot_core.xacro (robot description, xacro)
@@ -10,4 +10,11 @@
         <origin xyz="-0.1 0 0"/>
     </joint>
+    <joint name="base_footprint_joint" type="fixed">
+        <parent link="base_link"/>
+        <child link="base_footprint"/>
+        <origin xyz="0 0 -0.025"/>
+    </joint>
+    <link name="base_footprint">
+    </link>
  <!-- chassis link -->
     <link name="chassis">
